Commit message: Update the ATHLETE URDF joint limits to match the T12 model

File: urdf/TriATHLETE/urdf/TriATHLETE.URDF (robot description, URDF)
Before this commit: robot TriATHLETE, 31 links, 30 joints
Joints:
- joint AP1: limit effort=0 velocity=0 -> lower=-2.0944 upper=2.0944 effort=0 velocity=0
- joint AP2: limit effort=0 velocity=0 -> lower=-2.0944 upper=2.0944 effort=0 velocity=0
- joint AP3: limit effort=0 velocity=0 -> lower=-2.0944 upper=2.0944 effort=0 velocity=0
- joint AR1: limit effort=0 velocity=0 -> lower=-3.1416 upper=3.1416 effort=0 velocity=0
- joint AR2: limit effort=0 velocity=0 -> lower=-3.1416 upper=3.1416 effort=0 velocity=0
- joint AR3: limit effort=0 velocity=0 -> lower=-3.1416 upper=3.1416 effort=0 velocity=0
- joint HP1: limit effort=0 velocity=0 -> lower=-1.9199 upper=1.5708 effort=0 velocity=0
- joint HP2: limit effort=0 velocity=0 -> lower=-1.9199 upper=1.5708 effort=0 velocity=0
- joint HP3: limit effort=0 velocity=0 -> lower=-1.9199 upper=1.5708 effort=0 velocity=0
- joint HY1: limit effort=0 velocity=0 -> lower=-3.1416 upper=3.1416 effort=0 velocity=0
- joint HY2: limit effort=0 velocity=0 -> lower=-3.1416 upper=3.1416 effort=0 velocity=0
- joint HY3: limit effort=0 velocity=0 -> lower=-3.1416 upper=3.1416 effort=0 velocity=0
- joint KP1: limit effort=0 velocity=0 -> lower=-1.9199 upper=3.1416 effort=0 velocity=0
- joint KP2: limit effort=0 velocity=0 -> lower=-1.9199 upper=3.1416 effort=0 velocity=0
- joint KP3: limit effort=0 velocity=0 -> lower=-1.9199 upper=3.1416 effort=0 velocity=0
- joint KR1: limit effort=0 velocity=0 -> lower=-3.1416 upper=3.1416 effort=0 velocity=0
- joint KR2: limit effort=0 velocity=0 -> lower=-3.1416 upper=3.1416 effort=0 velocity=0
- joint KR3: limit effort=0 velocity=0 -> lower=-3.1416 upper=3.1416 effort=0 velocity=0

File: urdf/TriATHLETE_Climbing/urdf/TriATHLETE.URDF (robot description, URDF)
Before this commit: robot TriATHLETE, 28 links, 27 joints
Joints:
- joint AP1: limit effort=0 velocity=0 -> lower=-2.0944 upper=2.0944 effort=0 velocity=0
- joint AP2: limit effort=0 velocity=0 -> lower=-2.0944 upper=2.0944 effort=0 velocity=0
- joint AP3: limit effort=0 velocity=0 -> lower=-2.0944 upper=2.0944 effort=0 velocity=0
- joint AR1: limit effort=0 velocity=0 -> lower=-3.1416 upper=3.1416 effort=0 velocity=0
- joint AR2: limit effort=0 velocity=0 -> lower=-3.1416 upper=3.1416 effort=0 velocity=0
- joint AR3: limit effort=0 velocity=0 -> lower=-3.1416 upper=3.1416 effort=0 velocity=0
- joint HP1: limit effort=0 velocity=0 -> lower=-1.9199 upper=1.5708 effort=0 velocity=0
- joint HP2: limit effort=0 velocity=0 -> lower=-1.9199 upper=1.5708 effort=0 velocity=0
- joint HP3: limit effort=0 velocity=0 -> lower=-1.9199 upper=1.5708 effort=0 velocity=0
- joint HY1: limit effort=0 velocity=0 -> lower=-3.1416 upper=3.1416 effort=0 velocity=0
- joint HY2: limit effort=0 velocity=0 -> lower=-3.1416 upper=3.1416 effort=0 velocity=0
- joint HY3: limit effort=0 velocity=0 -> lower=-3.1416 upper=3.1416 effort=0 velocity=0
- joint KP1: limit effort=0 velocity=0 -> lower=-1.9199 upper=3.1416 effort=0 velocity=0
- joint KP2: limit effort=0 velocity=0 -> lower=-1.9199 upper=3.1416 effort=0 velocity=0
- joint KP3: limit effort=0 velocity=0 -> lower=-1.9199 upper=3.1416 effort=0 velocity=0
- joint KR1: limit effort=0 velocity=0 -> lower=-3.1416 upper=3.1416 effort=0 velocity=0
- joint KR2: limit effort=0 velocity=0 -> lower=-3.1416 upper=3.1416 effort=0 velocity=0
- joint KR3: limit effort=0 velocity=0 -> lower=-3.1416 upper=3.1416 effort=0 velocity=0

Commit message: Add prismatic joint limits

File: urdf/TriATHLETE/urdf/TriATHLETE.URDF (robot description, URDF)
Before this commit: robot TriATHLETE, 31 links, 30 joints
Joints:
- joint TC1A: limit effort=0 velocity=0 -> lower=0 upper=0.065 effort=0 velocity=0
- joint TC1B: limit effort=0 velocity=0 -> lower=0 upper=0.065 effort=0 velocity=0
- joint TC2A: limit effort=0 velocity=0 -> lower=0 upper=0.065 effort=0 velocity=0
- joint TC2B: limit effort=0 velocity=0 -> lower=0 upper=0.065 effort=0 velocity=0
- joint TC3A: limit effort=0 velocity=0 -> lower=0 upper=0.065 effort=0 velocity=0
- joint TC3B: limit effort=0 velocity=0 -> lower=0 upper=0.065 effort=0 velocity=0

File: urdf/TriATHLETE_Climbing/urdf/TriATHLETE.URDF (robot description, URDF)
Before this commit: robot TriATHLETE, 28 links, 27 joints
Joints:
- joint TC1A: axis 1 0 0 -> 0 -1 0; limit effort=0 velocity=0 -> lower=0 upper=0.065 effort=0 velocity=0
- joint TC1B: axis -1 0 0 -> 0 1 0; limit effort=0 velocity=0 -> lower=0 upper=0.065 effort=0 velocity=0
- joint TC2A: axis 1 0 0 -> 0 -1 0; limit effort=0 velocity=0 -> lower=0 upper=0.065 effort=0 velocity=0
- joint TC2B: axis -1 0 0 -> 0 1 0; limit effort=0 velocity=0 -> lower=0 upper=0.065 effort=0 velocity=0
- joint TC3A: axis 1 0 0 -> 0 -1 0; limit effort=0 velocity=0 -> lower=0 upper=0.065 effort=0 velocity=0
- joint TC3B: axis -1 0 0 -> 0 1 0; limit effort=0 velocity=0 -> lower=0 upper=0.065 effort=0 velocity=0
