Commit message: Make adjustments to the TriATHLETE Climbing robot to load the models from the proper package

File: urdf/TriATHLETE_Climbing/urdf/TriATHLETE.URDF (robot description, URDF)
Before this commit: robot TriATHLETE, 28 links, 27 joints
Links:
- link Ankle1: geometry collision mesh filename=package://TriATHLETE_Climbing/meshes/Ankle1.STL; visual mesh filename=package://TriATHLETE_Climbing/meshes/Ankle1.STL
- link Ankle2: geometry collision mesh filename=package://TriATHLETE_Climbing/meshes/Ankle2.STL; visual mesh filename=package://TriATHLETE_Climbing/meshes/Ankle2.STL
- link Ankle3: geometry collision mesh filename=package://TriATHLETE_Climbing/meshes/Ankle3.STL; visual mesh filename=package://TriATHLETE_Climbing/meshes/Ankle3.STL
- link Body: geometry collision mesh filename=package://TriATHLETE_Climbing/meshes/Body.STL; visual mesh filename=package://TriATHLETE_Climbing/meshes/Body.STL
- link Foot1: geometry collision mesh filename=package://TriATHLETE_Climbing/meshes/Foot1.STL; visual mesh filename=package://TriATHLETE_Climbing/meshes/Foot1.STL
- link Foot2: geometry collision mesh filename=package://TriATHLETE_Climbing/meshes/Foot2.STL; visual mesh filename=package://TriATHLETE_Climbing/meshes/Foot2.STL
- link Foot3: geometry collision mesh filename=package://TriATHLETE_Climbing/meshes/Foot3.STL; visual mesh filename=package://TriATHLETE_Climbing/meshes/Foot3.STL
- link Hip1: geometry collision mesh filename=package://TriATHLETE_Climbing/meshes/Hip1.STL; visual mesh filename=package://TriATHLETE_Climbing/meshes/Hip1.STL
- link Hip2: geometry collision mesh filename=package://TriATHLETE_Climbing/meshes/Hip2.STL; visual mesh filename=package://TriATHLETE_Climbing/meshes/Hip2.STL
- link Hip3: geometry collision mesh filename=package://TriATHLETE_Climbing/meshes/Hip3.STL; visual mesh filename=package://TriATHLETE_Climbing/meshes/Hip3.STL
- link Knee1: geometry collision mesh filename=package://TriATHLETE_Climbing/meshes/Knee1.STL; visual mesh filename=package://TriATHLETE_Climbing/meshes/Knee1.STL
- link Knee2: geometry collision mesh filename=package://TriATHLETE_Climbing/meshes/Knee2.STL; visual mesh filename=package://TriATHLETE_Climbing/meshes/Knee2.STL
- link Knee3: geometry collision mesh filename=package://TriATHLETE_Climbing/meshes/Knee3.STL; visual mesh filename=package://TriATHLETE_Climbing/meshes/Knee3.STL
- link Shin1: geometry collision mesh filename=package://TriATHLETE_Climbing/meshes/Shin1.STL; visual mesh filename=package://TriATHLETE_Climbing/meshes/Shin1.STL
- link Shin2: geometry collision mesh filename=package://TriATHLETE_Climbing/meshes/Shin2.STL; visual mesh filename=package://TriATHLETE_Climbing/meshes/Shin2.STL
- link Shin3: geometry collision mesh filename=package://TriATHLETE_Climbing/meshes/Shin3.STL; visual mesh filename=package://TriATHLETE_Climbing/meshes/Shin3.STL
- link Thigh1: geometry collision mesh filename=package://TriATHLETE_Climbing/meshes/Thigh1.STL; visual mesh filename=package://TriATHLETE_Climbing/meshes/Thigh1.STL
- link Thigh2: geometry collision mesh filename=package://TriATHLETE_Climbing/meshes/Thigh2.STL; visual mesh filename=package://TriATHLETE_Climbing/meshes/Thigh2.STL
- link Thigh3: geometry collision mesh filename=package://TriATHLETE_Climbing/meshes/Thigh3.STL; visual mesh filename=package://TriATHLETE_Climbing/meshes/Thigh3.STL
- link ToolCam1: geometry collision mesh filename=package://TriATHLETE_Climbing/meshes/ToolCam1.STL; visual mesh filename=package://TriATHLETE_Climbing/meshes/ToolCam1.STL
- link ToolCam2: geometry collision mesh filename=package://TriATHLETE_Climbing/meshes/ToolCam2.STL; visual mesh filename=package://TriATHLETE_Climbing/meshes/ToolCam2.STL
- link ToolCam3: geometry collision mesh filename=package://TriATHLETE_Climbing/meshes/ToolCam3.STL; visual mesh filename=package://TriATHLETE_Climbing/meshes/ToolCam3.STL
- link ToolClamp1A: geometry collision mesh filename=package://TriATHLETE_Climbing/meshes/ToolClamp1A.STL; visual mesh filename=package://TriATHLETE_Climbing/meshes/ToolClamp1A.STL
- link ToolClamp1B: geometry collision mesh filename=package://TriATHLETE_Climbing/meshes/ToolClamp1B.STL; visual mesh filename=package://TriATHLETE_Climbing/meshes/ToolClamp1B.STL
- link ToolClamp2A: geometry collision mesh filename=package://TriATHLETE_Climbing/meshes/ToolClamp2A.STL; visual mesh filename=package://TriATHLETE_Climbing/meshes/ToolClamp2A.STL
- link ToolClamp2B: geometry collision mesh filename=package://TriATHLETE_Climbing/meshes/ToolClamp2B.STL; visual mesh filename=package://TriATHLETE_Climbing/meshes/ToolClamp2B.STL
- link ToolClamp3A: geometry collision mesh filename=package://TriATHLETE_Climbing/meshes/ToolClamp3A.STL; visual mesh filename=package://TriATHLETE_Climbing/meshes/ToolClamp3A.STL
- link ToolClamp3B: geometry collision mesh filename=package://TriATHLETE_Climbing/meshes/ToolClamp3B.STL; visual mesh filename=package://TriATHLETE_Climbing/meshes/ToolClamp3B.STL
Joints:
- joint TC1A: limit lower=0 upper=0.065 effort=0 velocity=0 -> lower=0 upper=0.035 effort=0 velocity=0
- joint TC1B: limit lower=0 upper=0.065 effort=0 velocity=0 -> lower=0 upper=0.035 effort=0 velocity=0
- joint TC2A: limit lower=0 upper=0.065 effort=0 velocity=0 -> lower=0 upper=0.035 effort=0 velocity=0
- joint TC2B: limit lower=0 upper=0.065 effort=0 velocity=0 -> lower=0 upper=0.035 effort=0 velocity=0
- joint TC3A: limit lower=0 upper=0.065 effort=0 velocity=0 -> lower=0 upper=0.035 effort=0 velocity=0
- joint TC3B: limit lower=0 upper=0.065 effort=0 velocity=0 -> lower=0 upper=0.035 effort=0 velocity=0
