Commit message: Invert the joints

File: urdf/T12/urdf/T12_flipped.URDF (robot description, URDF)
Before this commit: robot T12, 37 links, 36 joints
Joints:
- joint AP1: axis 0 0 1 -> 0 0 -1
- joint AP2: axis 0 0 1 -> 0 0 -1
- joint AP3: axis 0 0 1 -> 0 0 -1
- joint AP4: axis 0 0 1 -> 0 0 -1
- joint AP5: axis 0 0 1 -> 0 0 -1
- joint AP6: axis 0 0 1 -> 0 0 -1
- joint AR1: axis 0 0 1 -> 0 0 -1
- joint AR2: axis 0 0 1 -> 0 0 -1
- joint AR3: axis 0 0 1 -> 0 0 -1
- joint AR4: axis 0 0 1 -> 0 0 -1
- joint AR5: axis 0 0 1 -> 0 0 -1
- joint AR6: axis 0 0 1 -> 0 0 -1
- joint HP1: axis 0 0 1 -> 0 0 -1
- joint HP2: axis 0 0 1 -> 0 0 -1
- joint HP3: axis 0 0 1 -> 0 0 -1
- joint HP4: axis 0 0 1 -> 0 0 -1
- joint HP5: axis 0 0 1 -> 0 0 -1
- joint HP6: axis 0 0 1 -> 0 0 -1
- joint HY1: axis 0 0 1 -> 0 0 -1
- joint HY2: axis 0 0 1 -> 0 0 -1
- joint HY3: axis 0 0 1 -> 0 0 -1
- joint HY4: axis 0 0 1 -> 0 0 -1
- joint HY5: axis 0 0 1 -> 0 0 -1
- joint HY6: axis 0 0 1 -> 0 0 -1
- joint KP1: axis 0 0 1 -> 0 0 -1
- joint KP2: axis 0 0 1 -> 0 0 -1
- joint KP3: axis 0 0 1 -> 0 0 -1
- joint KP4: axis 0 0 1 -> 0 0 -1
- joint KP5: axis 0 0 1 -> 0 0 -1
- joint KP6: axis 0 0 1 -> 0 0 -1
- joint KR1: axis 0 0 1 -> 0 0 -1
- joint KR2: axis 0 0 1 -> 0 0 -1
- joint KR3: axis 0 0 1 -> 0 0 -1
- joint KR4: axis 0 0 1 -> 0 0 -1
- joint KR5: axis 0 0 1 -> 0 0 -1
- joint KR6: axis 0 0 1 -> 0 0 -1

File: urdf/TriATHLETE/urdf/TriATHLETE_flipped.URDF (robot description, URDF)
Before this commit: robot TriATHLETE, 31 links, 30 joints
Joints:
- joint AP1: axis 0 0 1 -> 0 0 -1
- joint AP2: axis 0 0 1 -> 0 0 -1
- joint AP3: axis 0 0 1 -> 0 0 -1
- joint AR1: axis 0 0 1 -> 0 0 -1
- joint AR2: axis 0 0 1 -> 0 0 -1
- joint AR3: axis 0 0 1 -> 0 0 -1
- joint HP1: axis 0 0 1 -> 0 0 -1
- joint HP2: axis 0 0 1 -> 0 0 -1
- joint HP3: axis 0 0 1 -> 0 0 -1
- joint HY1: axis 0 0 1 -> 0 0 -1
- joint HY2: axis 0 0 1 -> 0 0 -1
- joint HY3: axis 0 0 1 -> 0 0 -1
- joint KP1: axis 0 0 1 -> 0 0 -1
- joint KP2: axis 0 0 1 -> 0 0 -1
- joint KP3: axis 0 0 1 -> 0 0 -1
- joint KR1: axis 0 0 1 -> 0 0 -1
- joint KR2: axis 0 0 1 -> 0 0 -1
- joint KR3: axis 0 0 1 -> 0 0 -1

File: urdf/TriATHLETE_Climbing/urdf/TriATHLETE_flipped.URDF (robot description, URDF)
Before this commit: robot TriATHLETE, 28 links, 27 joints
Joints:
- joint AP1: axis 0 0 1 -> 0 0 -1
- joint AP2: axis 0 0 1 -> 0 0 -1
- joint AP3: axis 0 0 1 -> 0 0 -1
- joint AR1: axis 0 0 1 -> 0 0 -1
- joint AR2: axis 0 0 1 -> 0 0 -1
- joint AR3: axis 0 0 1 -> 0 0 -1
- joint HP1: axis 0 0 1 -> 0 0 -1
- joint HP2: axis 0 0 1 -> 0 0 -1
- joint HP3: axis 0 0 1 -> 0 0 -1
- joint HY1: axis 0 0 1 -> 0 0 -1
- joint HY2: axis 0 0 1 -> 0 0 -1
- joint HY3: axis 0 0 1 -> 0 0 -1
- joint KP1: axis 0 0 1 -> 0 0 -1
- joint KP2: axis 0 0 1 -> 0 0 -1
- joint KP3: axis 0 0 1 -> 0 0 -1
- joint KR1: axis 0 0 1 -> 0 0 -1
- joint KR2: axis 0 0 1 -> 0 0 -1
- joint KR3: axis 0 0 1 -> 0 0 -1
