Commit message: Make example URDF paths relative

File: urdf/T12/urdf/T12.URDF (robot description, URDF)
Before this commit: robot T12, 37 links, 36 joints
Links:
- link Ankle1: geometry collision mesh filename=../meshes/Ankle1.STL; visual mesh filename=../meshes/Ankle1.STL
- link Ankle2: geometry collision mesh filename=../meshes/Ankle2.STL; visual mesh filename=../meshes/Ankle2.STL
- link Ankle3: geometry collision mesh filename=../meshes/Ankle3.STL; visual mesh filename=../meshes/Ankle3.STL
- link Ankle4: geometry collision mesh filename=../meshes/Ankle4.STL; visual mesh filename=../meshes/Ankle4.STL
- link Ankle5: geometry collision mesh filename=../meshes/Ankle5.STL; visual mesh filename=../meshes/Ankle5.STL
- link Ankle6: geometry collision mesh filename=../meshes/Ankle6.STL; visual mesh filename=../meshes/Ankle6.STL
- link Body: geometry collision mesh filename=../meshes/Body.STL; visual mesh filename=../meshes/Body.STL
- link Foot1: geometry collision mesh filename=../meshes/Foot1.STL; visual mesh filename=../meshes/Foot1.STL
- link Foot2: geometry collision mesh filename=../meshes/Foot2.STL; visual mesh filename=../meshes/Foot2.STL
- link Foot3: geometry collision mesh filename=../meshes/Foot3.STL; visual mesh filename=../meshes/Foot3.STL
- link Foot4: geometry collision mesh filename=../meshes/Foot4.STL; visual mesh filename=../meshes/Foot4.STL
- link Foot5: geometry collision mesh filename=../meshes/Foot5.STL; visual mesh filename=../meshes/Foot5.STL
- link Foot6: geometry collision mesh filename=../meshes/Foot6.STL; visual mesh filename=../meshes/Foot6.STL
- link Hip1: geometry collision mesh filename=../meshes/Hip1.STL; visual mesh filename=../meshes/Hip1.STL
- link Hip2: geometry collision mesh filename=../meshes/Hip2.STL; visual mesh filename=../meshes/Hip2.STL
- link Hip3: geometry collision mesh filename=../meshes/Hip3.STL; visual mesh filename=../meshes/Hip3.STL
- link Hip4: geometry collision mesh filename=../meshes/Hip4.STL; visual mesh filename=../meshes/Hip4.STL
- link Hip5: geometry collision mesh filename=../meshes/Hip5.STL; visual mesh filename=../meshes/Hip5.STL
- link Hip6: geometry collision mesh filename=../meshes/Hip6.STL; visual mesh filename=../meshes/Hip6.STL
- link Knee1: geometry collision mesh filename=../meshes/Knee1.STL; visual mesh filename=../meshes/Knee1.STL
- link Knee2: geometry collision mesh filename=../meshes/Knee2.STL; visual mesh filename=../meshes/Knee2.STL
- link Knee3: geometry collision mesh filename=../meshes/Knee3.STL; visual mesh filename=../meshes/Knee3.STL
- link Knee4: geometry collision mesh filename=../meshes/Knee4.STL; visual mesh filename=../meshes/Knee4.STL
- link Knee5: geometry collision mesh filename=../meshes/Knee5.STL; visual mesh filename=../meshes/Knee5.STL
- link Knee6: geometry collision mesh filename=../meshes/Knee6.STL; visual mesh filename=../meshes/Knee6.STL
- link Shin1: geometry collision mesh filename=../meshes/Shin1.STL; visual mesh filename=../meshes/Shin1.STL
- link Shin2: geometry collision mesh filename=../meshes/Shin2.STL; visual mesh filename=../meshes/Shin2.STL
- link Shin3: geometry collision mesh filename=../meshes/Shin3.STL; visual mesh filename=../meshes/Shin3.STL
- link Shin4: geometry collision mesh filename=../meshes/Shin4.STL; visual mesh filename=../meshes/Shin4.STL
- link Shin5: geometry collision mesh filename=../meshes/Shin5.STL; visual mesh filename=../meshes/Shin5.STL
- link Shin6: geometry collision mesh filename=../meshes/Shin6.STL; visual mesh filename=../meshes/Shin6.STL
- link Thigh1: geometry collision mesh filename=../meshes/Thigh1.STL; visual mesh filename=../meshes/Thigh1.STL
- link Thigh2: geometry collision mesh filename=../meshes/Thigh2.STL; visual mesh filename=../meshes/Thigh2.STL
- link Thigh3: geometry collision mesh filename=../meshes/Thigh3.STL; visual mesh filename=../meshes/Thigh3.STL
- link Thigh4: geometry collision mesh filename=../meshes/Thigh4.STL; visual mesh filename=../meshes/Thigh4.STL
- link Thigh5: geometry collision mesh filename=../meshes/Thigh5.STL; visual mesh filename=../meshes/Thigh5.STL
- link Thigh6: geometry collision mesh filename=../meshes/Thigh6.STL; visual mesh filename=../meshes/Thigh6.STL

File: urdf/T12/urdf/T12_flipped.URDF (robot description, URDF)
Before this commit: robot T12, 37 links, 36 joints
Links:
- link Ankle1: geometry collision mesh filename=../meshes/Ankle1.STL; visual mesh filename=../meshes/Ankle1.STL
- link Ankle2: geometry collision mesh filename=../meshes/Ankle2.STL; visual mesh filename=../meshes/Ankle2.STL
- link Ankle3: geometry collision mesh filename=../meshes/Ankle3.STL; visual mesh filename=../meshes/Ankle3.STL
- link Ankle4: geometry collision mesh filename=../meshes/Ankle4.STL; visual mesh filename=../meshes/Ankle4.STL
- link Ankle5: geometry collision mesh filename=../meshes/Ankle5.STL; visual mesh filename=../meshes/Ankle5.STL
- link Ankle6: geometry collision mesh filename=../meshes/Ankle6.STL; visual mesh filename=../meshes/Ankle6.STL
- link Body: geometry collision mesh filename=../meshes/Body.STL; visual mesh filename=../meshes/Body.STL
- link Foot1: geometry collision mesh filename=../meshes/Foot1.STL; visual mesh filename=../meshes/Foot1.STL
- link Foot2: geometry collision mesh filename=../meshes/Foot2.STL; visual mesh filename=../meshes/Foot2.STL
- link Foot3: geometry collision mesh filename=../meshes/Foot3.STL; visual mesh filename=../meshes/Foot3.STL
- link Foot4: geometry collision mesh filename=../meshes/Foot4.STL; visual mesh filename=../meshes/Foot4.STL
- link Foot5: geometry collision mesh filename=../meshes/Foot5.STL; visual mesh filename=../meshes/Foot5.STL
- link Foot6: geometry collision mesh filename=../meshes/Foot6.STL; visual mesh filename=../meshes/Foot6.STL
- link Hip1: geometry collision mesh filename=../meshes/Hip1.STL; visual mesh filename=../meshes/Hip1.STL
- link Hip2: geometry collision mesh filename=../meshes/Hip2.STL; visual mesh filename=../meshes/Hip2.STL
- link Hip3: geometry collision mesh filename=../meshes/Hip3.STL; visual mesh filename=../meshes/Hip3.STL
- link Hip4: geometry collision mesh filename=../meshes/Hip4.STL; visual mesh filename=../meshes/Hip4.STL
- link Hip5: geometry collision mesh filename=../meshes/Hip5.STL; visual mesh filename=../meshes/Hip5.STL
- link Hip6: geometry collision mesh filename=../meshes/Hip6.STL; visual mesh filename=../meshes/Hip6.STL
- link Knee1: geometry collision mesh filename=../meshes/Knee1.STL; visual mesh filename=../meshes/Knee1.STL
- link Knee2: geometry collision mesh filename=../meshes/Knee2.STL; visual mesh filename=../meshes/Knee2.STL
- link Knee3: geometry collision mesh filename=../meshes/Knee3.STL; visual mesh filename=../meshes/Knee3.STL
- link Knee4: geometry collision mesh filename=../meshes/Knee4.STL; visual mesh filename=../meshes/Knee4.STL
- link Knee5: geometry collision mesh filename=../meshes/Knee5.STL; visual mesh filename=../meshes/Knee5.STL
- link Knee6: geometry collision mesh filename=../meshes/Knee6.STL; visual mesh filename=../meshes/Knee6.STL
- link Shin1: geometry collision mesh filename=../meshes/Shin1.STL; visual mesh filename=../meshes/Shin1.STL
- link Shin2: geometry collision mesh filename=../meshes/Shin2.STL; visual mesh filename=../meshes/Shin2.STL
- link Shin3: geometry collision mesh filename=../meshes/Shin3.STL; visual mesh filename=../meshes/Shin3.STL
- link Shin4: geometry collision mesh filename=../meshes/Shin4.STL; visual mesh filename=../meshes/Shin4.STL
- link Shin5: geometry collision mesh filename=../meshes/Shin5.STL; visual mesh filename=../meshes/Shin5.STL
- link Shin6: geometry collision mesh filename=../meshes/Shin6.STL; visual mesh filename=../meshes/Shin6.STL
- link Thigh1: geometry collision mesh filename=../meshes/Thigh1.STL; visual mesh filename=../meshes/Thigh1.STL
- link Thigh2: geometry collision mesh filename=../meshes/Thigh2.STL; visual mesh filename=../meshes/Thigh2.STL
- link Thigh3: geometry collision mesh filename=../meshes/Thigh3.STL; visual mesh filename=../meshes/Thigh3.STL
- link Thigh4: geometry collision mesh filename=../meshes/Thigh4.STL; visual mesh filename=../meshes/Thigh4.STL
- link Thigh5: geometry collision mesh filename=../meshes/Thigh5.STL; visual mesh filename=../meshes/Thigh5.STL
- link Thigh6: geometry collision mesh filename=../meshes/Thigh6.STL; visual mesh filename=../meshes/Thigh6.STL

File: urdf/TriATHLETE/urdf/TriATHLETE.URDF (robot description, URDF)
Before this commit: robot TriATHLETE, 31 links, 30 joints
Links:
- link Ankle1: geometry collision mesh filename=../meshes/Ankle1.STL; visual mesh filename=../meshes/Ankle1.STL
- link Ankle2: geometry collision mesh filename=../meshes/Ankle2.STL; visual mesh filename=../meshes/Ankle2.STL
- link Ankle3: geometry collision mesh filename=../meshes/Ankle3.STL; visual mesh filename=../meshes/Ankle3.STL
- link Body: geometry collision mesh filename=../meshes/Body.STL; visual mesh filename=../meshes/Body.STL
- link Foot1: geometry collision mesh filename=../meshes/Foot1.STL; visual mesh filename=../meshes/Foot1.STL
- link Foot2: geometry collision mesh filename=../meshes/Foot2.STL; visual mesh filename=../meshes/Foot2.STL
- link Foot3: geometry collision mesh filename=../meshes/Foot3.STL; visual mesh filename=../meshes/Foot3.STL
- link Hip1: geometry collision mesh filename=../meshes/Hip1.STL; visual mesh filename=../meshes/Hip1.STL
- link Hip2: geometry collision mesh filename=../meshes/Hip2.STL; visual mesh filename=../meshes/Hip2.STL
- link Hip3: geometry collision mesh filename=../meshes/Hip3.STL; visual mesh filename=../meshes/Hip3.STL
- link Knee1: geometry collision mesh filename=../meshes/Knee1.STL; visual mesh filename=../meshes/Knee1.STL
- link Knee2: geometry collision mesh filename=../meshes/Knee2.STL; visual mesh filename=../meshes/Knee2.STL
- link Knee3: geometry collision mesh filename=../meshes/Knee3.STL; visual mesh filename=../meshes/Knee3.STL
- link Shin1: geometry collision mesh filename=../meshes/Shin1.STL; visual mesh filename=../meshes/Shin1.STL
- link Shin2: geometry collision mesh filename=../meshes/Shin2.STL; visual mesh filename=../meshes/Shin2.STL
- link Shin3: geometry collision mesh filename=../meshes/Shin3.STL; visual mesh filename=../meshes/Shin3.STL
- link Thigh1: geometry collision mesh filename=../meshes/Thigh1.STL; visual mesh filename=../meshes/Thigh1.STL
- link Thigh2: geometry collision mesh filename=../meshes/Thigh2.STL; visual mesh filename=../meshes/Thigh2.STL
- link Thigh3: geometry collision mesh filename=../meshes/Thigh3.STL; visual mesh filename=../meshes/Thigh3.STL
- link ToolCam1: geometry collision mesh filename=../meshes/ToolCam1.STL; visual mesh filename=../meshes/ToolCam1.STL
- link ToolCam2: geometry collision mesh filename=../meshes/ToolCam2.STL; visual mesh filename=../meshes/ToolCam2.STL
- link ToolCam3: geometry collision mesh filename=../meshes/ToolCam3.STL; visual mesh filename=../meshes/ToolCam3.STL
- link ToolClamp1A: geometry collision mesh filename=../meshes/ToolClamp1A.STL; visual mesh filename=../meshes/ToolClamp1A.STL
- link ToolClamp1B: geometry collision mesh filename=../meshes/ToolClamp1B.STL; visual mesh filename=../meshes/ToolClamp1B.STL
- link ToolClamp2A: geometry collision mesh filename=../meshes/ToolClamp2A.STL; visual mesh filename=../meshes/ToolClamp2A.STL
- link ToolClamp2B: geometry collision mesh filename=../meshes/ToolClamp2B.STL; visual mesh filename=../meshes/ToolClamp2B.STL
- link ToolClamp3A: geometry collision mesh filename=../meshes/ToolClamp3A.STL; visual mesh filename=../meshes/ToolClamp3A.STL
- link ToolClamp3B: geometry collision mesh filename=../meshes/ToolClamp3B.STL; visual mesh filename=../meshes/ToolClamp3B.STL
- link Wheel1: geometry collision mesh filename=../meshes/Wheel1.STL; visual mesh filename=../meshes/Wheel1.STL
- link Wheel2: geometry collision mesh filename=../meshes/Wheel2.STL; visual mesh filename=../meshes/Wheel2.STL
- link Wheel3: geometry collision mesh filename=../meshes/Wheel3.STL; visual mesh filename=../meshes/Wheel3.STL

File: urdf/TriATHLETE/urdf/TriATHLETE_flipped.URDF (robot description, URDF)
Before this commit: robot TriATHLETE, 31 links, 30 joints
Links:
- link Ankle1: geometry collision mesh filename=../meshes/Ankle1.STL; visual mesh filename=../meshes/Ankle1.STL
- link Ankle2: geometry collision mesh filename=../meshes/Ankle2.STL; visual mesh filename=../meshes/Ankle2.STL
- link Ankle3: geometry collision mesh filename=../meshes/Ankle3.STL; visual mesh filename=../meshes/Ankle3.STL
- link Body: geometry collision mesh filename=../meshes/Body.STL; visual mesh filename=../meshes/Body.STL
- link Foot1: geometry collision mesh filename=../meshes/Foot1.STL; visual mesh filename=../meshes/Foot1.STL
- link Foot2: geometry collision mesh filename=../meshes/Foot2.STL; visual mesh filename=../meshes/Foot2.STL
- link Foot3: geometry collision mesh filename=../meshes/Foot3.STL; visual mesh filename=../meshes/Foot3.STL
- link Hip1: geometry collision mesh filename=../meshes/Hip1.STL; visual mesh filename=../meshes/Hip1.STL
- link Hip2: geometry collision mesh filename=../meshes/Hip2.STL; visual mesh filename=../meshes/Hip2.STL
- link Hip3: geometry collision mesh filename=../meshes/Hip3.STL; visual mesh filename=../meshes/Hip3.STL
- link Knee1: geometry collision mesh filename=../meshes/Knee1.STL; visual mesh filename=../meshes/Knee1.STL
- link Knee2: geometry collision mesh filename=../meshes/Knee2.STL; visual mesh filename=../meshes/Knee2.STL
- link Knee3: geometry collision mesh filename=../meshes/Knee3.STL; visual mesh filename=../meshes/Knee3.STL
- link Shin1: geometry collision mesh filename=../meshes/Shin1.STL; visual mesh filename=../meshes/Shin1.STL
- link Shin2: geometry collision mesh filename=../meshes/Shin2.STL; visual mesh filename=../meshes/Shin2.STL
- link Shin3: geometry collision mesh filename=../meshes/Shin3.STL; visual mesh filename=../meshes/Shin3.STL
- link Thigh1: geometry collision mesh filename=../meshes/Thigh1.STL; visual mesh filename=../meshes/Thigh1.STL
- link Thigh2: geometry collision mesh filename=../meshes/Thigh2.STL; visual mesh filename=../meshes/Thigh2.STL
- link Thigh3: geometry collision mesh filename=../meshes/Thigh3.STL; visual mesh filename=../meshes/Thigh3.STL
- link ToolCam1: geometry collision mesh filename=../meshes/ToolCam1.STL; visual mesh filename=../meshes/ToolCam1.STL
- link ToolCam2: geometry collision mesh filename=../meshes/ToolCam2.STL; visual mesh filename=../meshes/ToolCam2.STL
- link ToolCam3: geometry collision mesh filename=../meshes/ToolCam3.STL; visual mesh filename=../meshes/ToolCam3.STL
- link ToolClamp1A: geometry collision mesh filename=../meshes/ToolClamp1A.STL; visual mesh filename=../meshes/ToolClamp1A.STL
- link ToolClamp1B: geometry collision mesh filename=../meshes/ToolClamp1B.STL; visual mesh filename=../meshes/ToolClamp1B.STL
- link ToolClamp2A: geometry collision mesh filename=../meshes/ToolClamp2A.STL; visual mesh filename=../meshes/ToolClamp2A.STL
- link ToolClamp2B: geometry collision mesh filename=../meshes/ToolClamp2B.STL; visual mesh filename=../meshes/ToolClamp2B.STL
- link ToolClamp3A: geometry collision mesh filename=../meshes/ToolClamp3A.STL; visual mesh filename=../meshes/ToolClamp3A.STL
- link ToolClamp3B: geometry collision mesh filename=../meshes/ToolClamp3B.STL; visual mesh filename=../meshes/ToolClamp3B.STL
- link Wheel1: geometry collision mesh filename=../meshes/Wheel1.STL; visual mesh filename=../meshes/Wheel1.STL
- link Wheel2: geometry collision mesh filename=../meshes/Wheel2.STL; visual mesh filename=../meshes/Wheel2.STL
- link Wheel3: geometry collision mesh filename=../meshes/Wheel3.STL; visual mesh filename=../meshes/Wheel3.STL

File: urdf/TriATHLETE_Climbing/urdf/TriATHLETE.URDF (robot description, URDF)
Before this commit: robot TriATHLETE, 28 links, 27 joints
Links:
- link Ankle1: geometry collision mesh filename=../meshes/Ankle1.STL; visual mesh filename=../meshes/Ankle1.STL
- link Ankle2: geometry collision mesh filename=../meshes/Ankle2.STL; visual mesh filename=../meshes/Ankle2.STL
- link Ankle3: geometry collision mesh filename=../meshes/Ankle3.STL; visual mesh filename=../meshes/Ankle3.STL
- link Body: geometry collision mesh filename=../meshes/Body.STL; visual mesh filename=../meshes/Body.STL
- link Foot1: geometry collision mesh filename=../meshes/Foot1.STL; visual mesh filename=../meshes/Foot1.STL
- link Foot2: geometry collision mesh filename=../meshes/Foot2.STL; visual mesh filename=../meshes/Foot2.STL
- link Foot3: geometry collision mesh filename=../meshes/Foot3.STL; visual mesh filename=../meshes/Foot3.STL
- link Hip1: geometry collision mesh filename=../meshes/Hip1.STL; visual mesh filename=../meshes/Hip1.STL
- link Hip2: geometry collision mesh filename=../meshes/Hip2.STL; visual mesh filename=../meshes/Hip2.STL
- link Hip3: geometry collision mesh filename=../meshes/Hip3.STL; visual mesh filename=../meshes/Hip3.STL
- link Knee1: geometry collision mesh filename=../meshes/Knee1.STL; visual mesh filename=../meshes/Knee1.STL
- link Knee2: geometry collision mesh filename=../meshes/Knee2.STL; visual mesh filename=../meshes/Knee2.STL
- link Knee3: geometry collision mesh filename=../meshes/Knee3.STL; visual mesh filename=../meshes/Knee3.STL
- link Shin1: geometry collision mesh filename=../meshes/Shin1.STL; visual mesh filename=../meshes/Shin1.STL
- link Shin2: geometry collision mesh filename=../meshes/Shin2.STL; visual mesh filename=../meshes/Shin2.STL
- link Shin3: geometry collision mesh filename=../meshes/Shin3.STL; visual mesh filename=../meshes/Shin3.STL
- link Thigh1: geometry collision mesh filename=../meshes/Thigh1.STL; visual mesh filename=../meshes/Thigh1.STL
- link Thigh2: geometry collision mesh filename=../meshes/Thigh2.STL; visual mesh filename=../meshes/Thigh2.STL
- link Thigh3: geometry collision mesh filename=../meshes/Thigh3.STL; visual mesh filename=../meshes/Thigh3.STL
- link ToolCam1: geometry collision mesh filename=../meshes/ToolCam1.STL; visual mesh filename=../meshes/ToolCam1.STL
- link ToolCam2: geometry collision mesh filename=../meshes/ToolCam2.STL; visual mesh filename=../meshes/ToolCam2.STL
- link ToolCam3: geometry collision mesh filename=../meshes/ToolCam3.STL; visual mesh filename=../meshes/ToolCam3.STL
- link ToolClamp1A: geometry collision mesh filename=../meshes/ToolClamp1A.STL; visual mesh filename=../meshes/ToolClamp1A.STL
- link ToolClamp1B: geometry collision mesh filename=../meshes/ToolClamp1B.STL; visual mesh filename=../meshes/ToolClamp1B.STL
- link ToolClamp2A: geometry collision mesh filename=../meshes/ToolClamp2A.STL; visual mesh filename=../meshes/ToolClamp2A.STL
- link ToolClamp2B: geometry collision mesh filename=../meshes/ToolClamp2B.STL; visual mesh filename=../meshes/ToolClamp2B.STL
- link ToolClamp3A: geometry collision mesh filename=../meshes/ToolClamp3A.STL; visual mesh filename=../meshes/ToolClamp3A.STL
- link ToolClamp3B: geometry collision mesh filename=../meshes/ToolClamp3B.STL; visual mesh filename=../meshes/ToolClamp3B.STL

File: urdf/TriATHLETE_Climbing/urdf/TriATHLETE_flipped.URDF (robot description, URDF)
Before this commit: robot TriATHLETE, 28 links, 27 joints
Links:
- link Ankle1: geometry collision mesh filename=../meshes/Ankle1.STL; visual mesh filename=../meshes/Ankle1.STL
- link Ankle2: geometry collision mesh filename=../meshes/Ankle2.STL; visual mesh filename=../meshes/Ankle2.STL
- link Ankle3: geometry collision mesh filename=../meshes/Ankle3.STL; visual mesh filename=../meshes/Ankle3.STL
- link Body: geometry collision mesh filename=../meshes/Body.STL; visual mesh filename=../meshes/Body.STL
- link Foot1: geometry collision mesh filename=../meshes/Foot1.STL; visual mesh filename=../meshes/Foot1.STL
- link Foot2: geometry collision mesh filename=../meshes/Foot2.STL; visual mesh filename=../meshes/Foot2.STL
- link Foot3: geometry collision mesh filename=../meshes/Foot3.STL; visual mesh filename=../meshes/Foot3.STL
- link Hip1: geometry collision mesh filename=../meshes/Hip1.STL; visual mesh filename=../meshes/Hip1.STL
- link Hip2: geometry collision mesh filename=../meshes/Hip2.STL; visual mesh filename=../meshes/Hip2.STL
- link Hip3: geometry collision mesh filename=../meshes/Hip3.STL; visual mesh filename=../meshes/Hip3.STL
- link Knee1: geometry collision mesh filename=../meshes/Knee1.STL; visual mesh filename=../meshes/Knee1.STL
- link Knee2: geometry collision mesh filename=../meshes/Knee2.STL; visual mesh filename=../meshes/Knee2.STL
- link Knee3: geometry collision mesh filename=../meshes/Knee3.STL; visual mesh filename=../meshes/Knee3.STL
- link Shin1: geometry collision mesh filename=../meshes/Shin1.STL; visual mesh filename=../meshes/Shin1.STL
- link Shin2: geometry collision mesh filename=../meshes/Shin2.STL; visual mesh filename=../meshes/Shin2.STL
- link Shin3: geometry collision mesh filename=../meshes/Shin3.STL; visual mesh filename=../meshes/Shin3.STL
- link Thigh1: geometry collision mesh filename=../meshes/Thigh1.STL; visual mesh filename=../meshes/Thigh1.STL
- link Thigh2: geometry collision mesh filename=../meshes/Thigh2.STL; visual mesh filename=../meshes/Thigh2.STL
- link Thigh3: geometry collision mesh filename=../meshes/Thigh3.STL; visual mesh filename=../meshes/Thigh3.STL
- link ToolCam1: geometry collision mesh filename=../meshes/ToolCam1.STL; visual mesh filename=../meshes/ToolCam1.STL
- link ToolCam2: geometry collision mesh filename=../meshes/ToolCam2.STL; visual mesh filename=../meshes/ToolCam2.STL
- link ToolCam3: geometry collision mesh filename=../meshes/ToolCam3.STL; visual mesh filename=../meshes/ToolCam3.STL
- link ToolClamp1A: geometry collision mesh filename=../meshes/ToolClamp1A.STL; visual mesh filename=../meshes/ToolClamp1A.STL
- link ToolClamp1B: geometry collision mesh filename=../meshes/ToolClamp1B.STL; visual mesh filename=../meshes/ToolClamp1B.STL
- link ToolClamp2A: geometry collision mesh filename=../meshes/ToolClamp2A.STL; visual mesh filename=../meshes/ToolClamp2A.STL
- link ToolClamp2B: geometry collision mesh filename=../meshes/ToolClamp2B.STL; visual mesh filename=../meshes/ToolClamp2B.STL
- link ToolClamp3A: geometry collision mesh filename=../meshes/ToolClamp3A.STL; visual mesh filename=../meshes/ToolClamp3A.STL
- link ToolClamp3B: geometry collision mesh filename=../meshes/ToolClamp3B.STL; visual mesh filename=../meshes/ToolClamp3B.STL
